File: hardware/lupa.kicad_sch (KiCad schematic)
At the start: 74 parts, among them J1 LEVER, J10 LED_PWR, J11 MAX31865, J12 POWER, J13 PROG, J14 BOILER_SSR, J15 Screw_Terminal_01x01, J16 Mains, J17 Fill Solenoid, J18 Pump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

Commit message: Update BOM
Parts:
- C14: Farnell (none) -> 2610819
- C8: Farnell (none) -> 2614008
- DRL1, DRL2, DRL3, DRL4, LOGO2: now left out of the parts list
- F1: Farnell (none) -> 1829461
- J1, J10, J12, J19, J2, J3: Farnell (none) -> 3287572
- J11: Purchase Link (none) -> https://www.aliexpress.com/item/1005006704297164.html
- J14: Farnell (none) -> 3287588
- J4, J5, J6, J7: Farnell (none) -> 3287574
- J8, J9: Farnell (none) -> 3287578
- R16: Farnell (none) -> 1357899
- U1: LCSC (none) -> C328062
- U2: Farnell (none) -> 3870399
- U3, U4: Farnell (none) -> 4204024; Mouser (none) -> 769-AQH1213A
